File: JK-RFT Electrical/JK-RFT boards/JK-RFT-ELCT-01-01-01 USB-C breakout/JK-RFT-ELCT-01-01-01 USB-C breakout.kicad_sch (KiCad schematic)
At the start: 5 parts, among them J1 USB_C_Receptacle_USB2.0_16P, J2 Conn_01x04, U1 USBLC6-2SC6

Commit message: created JK-RFT-ELCT-01-01-01 USB C breakout board
Connections:
- net Di-: now reaches J1.A7 (D-), J1.B7 (D-), U1.1 (I/O1)
- net Di+: now reaches J1.A6 (D+), J1.B6 (D+), U1.3 (I/O2)
- net Do+: now reaches J2.4 (Pin_4), U1.4 (I/O2)
- net Do-: now reaches J2.3 (Pin_3), U1.6 (I/O1)
Changed lines of the file:
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@@
+		)
+	)
+	(label "Di-"
+		(at 85.09 69.85 0)
+		(effects
+			(font
+				(size 1.27 1.27)
+			)
+			(justify left bottom)
+		)
+	)
+	(label "Do-"
+		(at 110.49 69.85 0)
+		(effects
+			(font
+				(size 1.27 1.27)
+			)
+			(justify left bottom)
+		)
+	)
+	(label "Di+"
+		(at 85.09 72.39 0)
+		(effects
+			(font
+				(size 1.27 1.27)
+			)
+			(justify left bottom)
+		)
+	)
+	(label "Do+"
+		(at 110.49 72.39 0)
+		(effects
+			(font
+				(size 1.27 1.27)
+			)
+			(justify left bottom)
 		)
 	)
