File: JK-RFT Electrical/JK-RFT boards/JK-RFT-ELCT-01-02-01 Main PCB/JK-RFT-ELCT-01-02-01 Main PCB.kicad_sch (KiCad schematic)
At the start: 21 parts, among them J1 POWER, J10 E7, J11 E8, J12 E9, J13 E10, J14 PLUS, J15 MINUS, J16 MULTIPLY, J17 DIVIDE, J2 Handset SW, J3 SPK LED, J4 E1, J5 E2, J6 E3, J7 E4, J8 E5, J9 E6, U2 AA1, U3 AA2

Commit message: created main pcb layout, not routed yet
Parts:
- removed A1: RaspberryPi_Pico, Module:RaspberryPi_Pico_Common_Unspecified, symbol MCU_Module:RaspberryPi_Pico
- added A2: RaspberryPi_Pico, Module:RaspberryPi_Pico_Common_THT, symbol MCU_Module:RaspberryPi_Pico_Extensive
- added C1, C3, C5: 100nF, Capacitor_SMD:C_0603_1608Metric_Pad1.08x0.95mm_HandSolder, symbol Device:C_Small
- added C2, C4: 22uF, Capacitor_SMD:C_0805_2012Metric_Pad1.18x1.45mm_HandSolder, symbol Device:C_Small
- added C6: 10uF, Capacitor_SMD:C_0805_2012Metric_Pad1.18x1.45mm_HandSolder, symbol Device:C_Small
- added J18: DEBUG, Connector_JST:JST_XH_B4B-XH-A_1x04_P2.50mm_Vertical, symbol Connector:Conn_01x04_Pin
- added SW1: Reset, Button_Switch_THT:SW_PUSH_6mm, symbol Switch:SW_Push
- J1, J2, J3: footprint (none) -> Connector_JST:JST_XH_B2B-XH-A_1x02_P2.50mm_Vertical
- J10, J11, J12, J13, J4, J5, J6, J7, J8, J9: footprint (none) -> Connector_JST:JST_XH_B4B-XH-A_1x04_P2.50mm_Vertical
- J14: value PLUS -> +; footprint (none) -> Connector_JST:JST_XH_B2B-XH-A_1x02_P2.50mm_Vertical
- J15: value MINUS -> -; footprint (none) -> Connector_JST:JST_XH_B2B-XH-A_1x02_P2.50mm_Vertical
- J16: value MULTIPLY -> ×; footprint (none) -> Connector_JST:JST_XH_B2B-XH-A_1x02_P2.50mm_Vertical
- J17: value DIVIDE -> ÷; footprint (none) -> Connector_JST:JST_XH_B2B-XH-A_1x02_P2.50mm_Vertical
- U1: value ~ -> uSD reader; footprint (none) -> Connector_PinHeader_2.54mm:PinHeader_1x06_P2.54mm_Vertical
- U2, U3: footprint (none) -> MAX98357A AA module:MODULE_3006
Connections:
- net DIVIDE: now also A2.34 (GPIO28_ADC2)
- net ENSW: now also A2.21 (GPIO16)
- net GND: now also U2.2 (GND), U3.2 (GND), A2.13 (GND), A2.18 (GND), A2.23 (GND), A2.28 (GND), A2.3 (GND), A2.33 (AGND), A2.38 (GND), A2.8 (GND), A2.D2 (GND), C1.2, C2.2, C3.2, C4.2, C5.2, C6.2, J18.1 (Pin_1), SW1.1; no longer U2.6 (GND), U3.6 (GND)
- net HSSW: now also A2.1 (GPIO0)
- net MINUS: now also A2.31 (GPIO26_ADC0)
- net MULTIPLY: now also A2.32 (GPIO27_ADC1)
- net N0: now also A2.20 (GPIO15)
- net N1: now also A2.9 (GPIO6)
- net N2: now also A2.10 (GPIO7)
- net N3: now also A2.11 (GPIO8)
- net N4: now also A2.12 (GPIO9)
- net N5: now also A2.14 (GPIO10)
- net N6: now also A2.15 (GPIO11)
- net N7: now also A2.16 (GPIO12)
- net N8: now also A2.17 (GPIO13)
- net N9: now also A2.19 (GPIO14)
- net PLUS: now also A2.29 (GPIO22)
- net SPK LED: now also A2.2 (GPIO1)
- net VCC: now also U2.1 (VIN), U3.1 (VIN), A2.40 (VBUS), C1.1, C2.1, C3.1, C4.1; no longer U1.5 (VCC), U2.7 (VIN), U3.7 (VIN)
- net at U2.5 (DIN): now also U3.5 (DIN), A2.27 (GPIO21)
- net at U2.3 (SD): now also A2.22 (GPIO17); no longer U3.3 (DIN)
- net at U1.2 (CS): now also A2.7 (GPIO5)
- net at U1.3 (MOSI): now also A2.5 (GPIO3)
- net at U1.4 (SCK): now also A2.4 (GPIO2)
- net +3V3: now reaches U1.1 (3V3)
- net +3V3: now also A2.36 (3V3), C5.1, C6.1
- new net: A2.24 (GPIO18), U3.3 (SD)
- new net: A2.25 (GPIO19), U2.7 (LRC), U3.7 (LRC)
- new net: A2.26 (GPIO20), U2.6 (BCLK), U3.6 (BCLK)
- new net: A2.6 (GPIO4), U1.5 (MISO)
- new net RUN: A2.30 (RUN), J18.4 (Pin_4), SW1.2
- new net SWCLK: A2.D1 (SWCLK), J18.2 (Pin_2)
- new net SWDIO: A2.D3 (SWDIO), J18.3 (Pin_3)
- no-connect marks 5 -> 10
Other:
- moved on the sheet: J10, J11, J12, J13, J14, J15, J16, J17, J4, J5, J6, J7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

Commit message: finished main pcb
Parts:
- removed J18: DEBUG, Connector_JST:JST_XH_B4B-XH-A_1x04_P2.50mm_Vertical, symbol Connector:Conn_01x04_Pin
Connections:
- net SWCLK: no longer names the net of A2.D1 (SWCLK)
- net SWDIO: no longer names the net of A2.D3 (SWDIO)
- no-connect marks 10 -> 12
Changed lines of the file:
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@@
+	)
+	(no_connect
+		(at 165.1 66.04)
 	)
 	(no_connect
@@
 	)
 	(no_connect
+		(at 165.1 68.58)
+	)
+	(no_connect
 		(at 168.91 76.2)
 	)
@@
 	(wire
 		(pts
-			(xy 43.18 176.53) (xy 50.8 176.53)
-		)
-		(stroke
-			(width 0)
-			(type default)
-		)
-	)
-	(wire
-		(pts
 			(xy 81.28 149.86) (xy 81.28 154.94)
 		)
@@
 	(wire
 		(pts
-			(xy 43.18 168.91) (xy 45.72 168.91)
-		)
-		(stroke
-			(width 0)
-			(type default)
-		)
-	)
-	(wire
-		(pts
 			(xy 85.09 104.14) (xy 85.09 116.84)
 		)
@@
 	(wire
 		(pts
-			(xy 45.72 168.91) (xy 45.72 180.34)
-		)
-		(stroke
-			(width 0)
-			(type default)
-		)
-	)
-	(wire
-		(pts
 			(xy 80.01 71.12) (xy 80.01 76.2)
 		)
@@
 	(wire
 		(pts
-			(xy 43.18 171.45) (xy 50.8 171.45)
-		)
-		(stroke
-			(width 0)
-			(type default)
-		)
-	)
-	(wire
-		(pts
 			(xy 165.1 116.84) (xy 168.91 116.84)
 		)
@@
 		(pts
 			(xy 85.09 78.74) (xy 85.09 91.44)
-		)
-		(stroke
-			(width 0)
-			(type default)
-		)
-	)
-	(wire
-		(pts
-			(xy 43.18 173.99) (xy 50.8 173.99)
 		)
 		(stroke
@@
 		)
 	)
-	(label "RUN"
-		(at 50.8 176.53 0)
-		(effects
-			(font
-				(size 1.27 1.27)
-			)
-			(justify left bottom)
-		)
-	)
 	(label "N8"
 		(at 88.9 99.06 0)
@@
 		)
 	)
-	(label "SWCLK"
-		(at 50.8 171.45 0)
-		(effects
-			(font
-				(size 1.27 1.27)
-			)
-			(justify left bottom)
-		)
-	)
 	(label "DIVIDE"
 		(at 85.09 152.4 0)
@@
 		)
 	)
-	(label "SWDIO"
-		(at 50.8 173.99 0)
-		(effects
-			(font
-				(size 1.27 1.27)
-			)
-			(justify left bottom)
-		)
-	)
 	(label "RUN"
 		(at 137.16 29.21 0)
@@
 		)
 	)
-	(label "SWDIO"
-		(at 165.1 68.58 180)
-		(effects
-			(font
-				(size 1.27 1.27)
-			)
-			(justify right bottom)
-		)
-	)
 	(label "N3"
 		(at 50.8 73.66 0)
@@
 	(label "HSSW"
 		(at 165.1 81.28 180)
-		(effects
-			(font
-				(size 1.27 1.27)
-			)
-			(justify right bottom)
-		)
-	)
-	(label "SWCLK"
-		(at 165.1 66.04 180)
 		(effects
 			(font
@@
 	(symbol
 		(lib_id "power:GND")
-		(at 45.72 180.34 0)
-		(unit 1)
-		(exclude_from_sim no)
-		(in_bom yes)
-		(on_board yes)
-		(dnp no)
-		(fields_autoplaced yes)
-		(property "Reference" "#PWR020"
-			(at 45.72 186.69 0)
-			(effects
-				(font
-					(size 1.27 1.27)
-				)
-				(hide yes)
-			)
-		)
-		(property "Value" "GND"
-			(at 45.72 185.42 0)
-			(effects
-				(font
-					(size 1.27 1.27)
-				)
-			)
-		)
-		(property "Footprint" ""
-			(at 45.72 180.34 0)
-			(effects
-				(font
-					(size 1.27 1.27)
-				)
-				(hide yes)
-			)
-		)
-		(property "Datasheet" ""
-			(at 45.72 180.34 0)
-			(effects
-				(font
-					(size 1.27 1.27)
-				)
-				(hide yes)
-			)
-		)
-		(property "Description" "Power symbol creates a global label with name \"GND\" , ground"
-			(at 45.72 180.34 0)
-			(effects
-				(font
-					(size 1.27 1.27)
-				)
-				(hide yes)
-			)
-		)
-		(pin "1"
-		)
-		(instances
-			(project "JK-RFT-ELCT-01-02-01 Main PCB"
-				(path "/8875e8fa-6bed-4959-b229-7df4163389c9"
-					(reference "#PWR020")
-					(unit 1)
-				)
-			)
-		)
-	)
-	(symbol
-		(lib_id "power:GND")
 		(at 81.28 154.94 0)
 		(unit 1)
@@
 					(unit 1)
 				)
-			)
-		)
-	)
-	(symbol
-		(lib_id "Connector:Conn_01x04_Pin")
-		(at 38.1 171.45 0)
-		(unit 1)
-		(exclude_from_sim no)
-		(in_bom yes)
-		(on_board yes)
-		(dnp no)
-		(property "Reference" "J18"
-			(at 35.56 171.196 0)
-			(effects
-				(font
-					(size 1.27 1.27)
-				)
-			)
-		)
-		(property "Value" "DEBUG"
-			(at 34.036 173.736 0)
-			(effects
-				(font
-					(size 1.27 1.27)
-				)
-			)
-		)
-		(property "Footprint" "Connector_JST:JST_XH_B4B-XH-A_1x04_P2.50mm_Vertical"
-			(at 38.1 171.45 0)
-			(effects
-				(font
-					(size 1.27 1.27)
-				)
-				(hide yes)
-			)
-		)
-		(property "Datasheet" "~"
-			(at 38.1 171.45 0)
-			(effects
-				(font
-					(size 1.27 1.27)
-				)
-				(hide yes)
-			)
-		)
-		(property "Description" "Generic connector, single row, 01x04, script generated"
-			(at 38.1 171.45 0)
-			(effects
-				(font
-					(size 1.27 1.27)
-				)
-				(hide yes)
-			)
-		)
-		(pin "4"
-		)
-		(pin "3"
-		)
-		(pin "1"
-		)
-		(pin "2"
-		)
-		(instances
-			(project "JK-RFT-ELCT-01-02-01 Main PCB"
-				(path "/8875e8fa-6bed-4959-b229-7df4163389c9"
-					(reference "J18")
-					(unit 1)
-				)
