File: JK-RFT Electrical/JK-RFT boards/JK-RFT-ELCT-01-02-01 Main PCB/JK-RFT-ELCT-01-02-01 Main PCB.kicad_pcb (KiCad board)
At the start: 2 copper layers, 0 parts

Commit message: created main pcb layout, not routed yet
Parts:
- added A2: RaspberryPi_Pico, Module:RaspberryPi_Pico_Common_THT, F.Cu at (115.1, 93.2)
- added C1: 100nF, Capacitor_SMD:C_0603_1608Metric_Pad1.08x0.95mm_HandSolder, B.Cu at (182.3, 70.2)
- added C2: 22uF, Capacitor_SMD:C_0805_2012Metric_Pad1.18x1.45mm_HandSolder, B.Cu at (182.5, 72.3)
- added C3: 100nF, Capacitor_SMD:C_0603_1608Metric_Pad1.08x0.95mm_HandSolder, B.Cu at (171.1, 121.7)
- added C4: 22uF, Capacitor_SMD:C_0805_2012Metric_Pad1.18x1.45mm_HandSolder, B.Cu at (170.9, 119.3)
- added C5: 100nF, Capacitor_SMD:C_0603_1608Metric_Pad1.08x0.95mm_HandSolder, B.Cu at (189.1, 91.6)
- added C6: 10uF, Capacitor_SMD:C_0805_2012Metric_Pad1.18x1.45mm_HandSolder, B.Cu at (186.8, 91.8)
- added J1: POWER, Connector_JST:JST_XH_B2B-XH-A_1x02_P2.50mm_Vertical, F.Cu at (152.4, 59.2)
- added J10: E7, Connector_JST:JST_XH_B4B-XH-A_1x04_P2.50mm_Vertical, F.Cu at (155.4, 109.2)
- added J11: E8, Connector_JST:JST_XH_B4B-XH-A_1x04_P2.50mm_Vertical, F.Cu at (170.3, 109.2)
- added J12: E9, Connector_JST:JST_XH_B4B-XH-A_1x04_P2.50mm_Vertical, F.Cu at (125.5, 117.3)
- added J13: E10, Connector_JST:JST_XH_B4B-XH-A_1x04_P2.50mm_Vertical, F.Cu at (140.4, 117.3)
- added J14: +, Connector_JST:JST_XH_B2B-XH-A_1x02_P2.50mm_Vertical, F.Cu at (153.0, 126.2)
- added J15: -, Connector_JST:JST_XH_B2B-XH-A_1x02_P2.50mm_Vertical, F.Cu at (163.0, 126.2)
- added J16: ×, Connector_JST:JST_XH_B2B-XH-A_1x02_P2.50mm_Vertical, F.Cu at (153.0, 134.2)
- added J17: ÷, Connector_JST:JST_XH_B2B-XH-A_1x02_P2.50mm_Vertical, F.Cu at (163.0, 134.2)
- added J18: DEBUG, Connector_JST:JST_XH_B4B-XH-A_1x04_P2.50mm_Vertical, F.Cu at (140.0, 126.1)
- added J2: Handset SW, Connector_JST:JST_XH_B2B-XH-A_1x02_P2.50mm_Vertical, F.Cu at (146.8, 67.8)
- added J3: SPK LED, Connector_JST:JST_XH_B2B-XH-A_1x02_P2.50mm_Vertical, F.Cu at (158.2, 67.8)
- added J4: E1, Connector_JST:JST_XH_B4B-XH-A_1x04_P2.50mm_Vertical, F.Cu at (125.5, 101.1)
- added J5: E2, Connector_JST:JST_XH_B4B-XH-A_1x04_P2.50mm_Vertical, F.Cu at (140.4, 101.1)
- added J6: E3, Connector_JST:JST_XH_B4B-XH-A_1x04_P2.50mm_Vertical, F.Cu at (155.4, 101.1)
- added J7: E4, Connector_JST:JST_XH_B4B-XH-A_1x04_P2.50mm_Vertical, F.Cu at (170.3, 101.1)
- added J8: E5, Connector_JST:JST_XH_B4B-XH-A_1x04_P2.50mm_Vertical, F.Cu at (125.5, 109.2)
- added J9: E6, Connector_JST:JST_XH_B4B-XH-A_1x04_P2.50mm_Vertical, F.Cu at (140.4, 109.2)
- added SW1: Reset, Button_Switch_THT:SW_PUSH_6mm, F.Cu at (132.0, 69.1)
- added U1: uSD reader, Connector_PinHeader_2.54mm:PinHeader_1x06_P2.54mm_Vertical, F.Cu at (183.3, 90.8)
- added U2: AA1, MAX98357A AA module:MODULE_3006, F.Cu at (176.4, 68.5)
- added U3: AA2, MAX98357A AA module:MODULE_3006, F.Cu at (177.0, 123.2)
Routing:
- net /RUN: track 0.00 -> 6.50 mm
- added copper zone on In2.Cu, net +3V3
- added copper zone on In1.Cu, net GND
- added copper zone on B.Cu, net VCC
Other:
- board outline added: 90 x 90 mm
- copper layers 2 -> 4

Commit message: finished main pcb
Parts:
- removed J18: DEBUG, Connector_JST:JST_XH_B4B-XH-A_1x04_P2.50mm_Vertical
- added G***: LOGO, Documents:Spooderman footprint, F.Cu at (123.2, 125.3)
- added G***: LOGO, Documents:Spooderman footprint, F.Cu at (182.4, 83.9)
- added G***: LOGO, Documents:Spooderman footprint, F.Cu at (162.1, 64.3)
- added G***: LOGO, Documents:Spooderman footprint, F.Cu at (152.9, 117.1)
- added G***: LOGO, Documents:Spooderman footprint, F.Cu at (152.2, 67.2)
- added G***: LOGO, Documents:Spooderman footprint, F.Cu at (178.8, 108.3)
- added G***: LOGO, Documents:Spooderman footprint, F.Cu at (170.1, 85.3)
- added G***: LOGO, Documents:Spooderman footprint, F.Cu at (144.8, 68.5)
- added G***: LOGO, Documents:Spider logo 40x40, B.Cu at (132.7, 108.5)
- moved J2 66.8 mm to (140.0, 134.2)
- moved J3 61.2 mm to (140.0, 126.3)
- moved J12 47.7 mm to (170.3, 101.1)
- moved J6 34.0 mm to (125.5, 117.3)
- moved J13 31.0 mm to (170.3, 109.2)
- moved J7 29.9 mm to (140.4, 101.1)
- moved J5 17.0 mm to (125.5, 109.2)
- moved J11 15.0 mm to (155.4, 109.2)
- moved J8 15.0 mm to (140.4, 109.2)
- moved J10 8.09 mm to (155.4, 101.1)
- moved J9 8.09 mm to (140.4, 117.3)
- moved C3 2.53 mm to (170.2, 119.3)
- moved C4 2.19 mm to (170.4, 121.4)
- moved C5 2.14 mm to (188.1, 89.8), turned to 0 degrees
- moved C6 1.37 mm to (188.1, 92.0), turned to 0 degrees
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Routing:
- net /DIVIDE: track 0.00 -> 118.9 mm
- net /MINUS: track 0.00 -> 115.9 mm
- net /MULTIPLY: track 0.00 -> 108.6 mm
- net /PLUS: track 0.00 -> 106.1 mm
- net Net-(A2-GPIO21): track 0.00 -> 89.3 mm
- net Net-(A2-GPIO20): track 0.00 -> 81.5 mm
- net Net-(A2-GPIO2): track 0.00 -> 72.5 mm
- net Net-(A2-GPIO19): track 0.00 -> 71.5 mm
- net Net-(A2-GPIO3): track 0.00 -> 71.4 mm
- net Net-(A2-GPIO5): track 0.00 -> 70.3 mm
- net Net-(A2-GPIO18): track 0.00 -> 69.1 mm
- net Net-(A2-GPIO4): track 0.00 -> 59.9 mm
- net /HSSW: track 0.00 -> 58.5 mm
- net /SPK LED: track 0.00 -> 55.0 mm
- net /N3: track 0.00 -> 33.1 mm
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- added copper zone on F.Cu, net /ENSW

Commit message: added one piece is real
Parts:
- moved G*** 3.70 mm to (186.1, 83.8)
Other:
- board text added: "MAX98357A Module Audio Amplifier"
- board text added: "The One Piece... is REAL!"
